File: Verstaerkerplatine/Messplatine/Messplatine.kicad_sch (KiCad schematic)
At the start: 48 parts, among them J1 Conn_01x20_Socket, J14 Conn_01x20_Socket, J26 Conn_02x20_Odd_Even, U1 MCP6042, U10 KY-051, U11 ULN2003, U3 TMA0505D, U31 Powersupply, U4 CA3140, U5 AD623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

Commit message: added Jumpers for 3.3V and 5V from Raspberry Pi
Parts:
- added JP1, JP2: Jumper_2_Open, Connector_PinHeader_2.54mm:PinHeader_1x02_P2.54mm_Vertical, symbol Jumper:Jumper_2_Open
Connections:
- net +3.3V: now also JP1.1 (A)
- net +5V: now also JP2.2 (B)
- net -5V: now also C10.2; no longer C10.1
- net at C9.1, U3.5, U4.7 (V+): now also C10.1; no longer C10.2
- net at J26.1 (Pin_1): now also JP1.2 (B)
- net at J26.2 (Pin_2): now also JP2.1 (A)
- no-connect marks 39 -> 37

Commit message: introduced direct wire connections for CA3160 and INA219
Parts:
- added J2: Elektrometer_In, Connector_PinHeader_2.54mm:PinHeader_1x01_P2.54mm_Vertical, symbol Connector:Conn_01x01_Pin
- JP1, JP2: value Jumper_2_Open -> J_2_Open
Connections:
- net +3.3V: now also JP1.2 (B); no longer JP1.1 (A)
- net GND: now also J14.3 (Pin_3)
- net at J26.1 (Pin_1): now also JP1.1 (A); no longer JP1.2 (B)
- net Elektrometer_IN_+: no longer names the net of U4.3 (+)
- net Elektrometer_IN_+: now also J2.1 (Pin_1); no longer J14.3 (Pin_3)
- removed net StromSpannungsSensor_IN_+: J1.5 (Pin_5), J1.6 (Pin_6), U6.6
- removed net StromSpannungsSensor_IN_-: J1.3 (Pin_3), J1.4 (Pin_4), U6.5
- no-connect marks 37 -> 43
Other:
- moved on the sheet: JP1
